File: Research and Development/BMS/PCB Design/3.0 BMS/V3.2/BMS MK2.kicad_pcb (KiCad board)
At the start: 2 copper layers, 246.6 x 98.4 mm, 49 parts, among them J1 Conn_01x04_Socket, J2 Charger out, J3 PWR IN, J5 CHG IN, Q1 AO3400A, Q2 PN100, Q3 AO3407, Q4 AO3407, Q5 PN100, Q7 PN100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

Commit message: updated bms schem
fixed polarity on batteries, updated jst conns to XH, created footprints for them, tidied up and shrunk the board size, changed from using the ds18d20b to a 10k ntc thermistor for temperature control protection
Parts:
- removed B1, B2, B3, B4: ~, DCDC buck converter lm2596:18650 Batt 2S Holder
- removed J5: CHG IN, Connector_JST:JST_GH_SM04B-GHS-TB_1x04-1MP_P1.25mm_Horizontal
- removed U5: DS18B20, Package_TO_SOT_THT:TO-92_Inline
- added B5: ~, DCDC buck converter lm2596:18650 Batt 2S Holder, B.Cu at (71.6, 58.6)
- added B6: ~, DCDC buck converter lm2596:18650 Batt 2S Holder, B.Cu at (145.2, 135.6)
- added B7: ~, DCDC buck converter lm2596:18650 Batt 2S Holder, F.Cu at (145.1, 58.1)
- added B8: ~, DCDC buck converter lm2596:18650 Batt 2S Holder, F.Cu at (71.6, 135.7)
- added D3: ON LED, LED_SMD:LED_1206_3216Metric, F.Cu at (180.3, 97.0)
- added D4: CHG LED, LED_SMD:LED_1206_3216Metric, F.Cu at (203.6, 97.0)
- added DS1: WC1602A, Display:WC1602A, F.Cu at (-90.3, 14.7)
- added J2: B CHG IN, DCDC buck converter lm2596:kf1000 screw terminal, F.Cu at (209.5, 135.3)
- added J6: load chg in, DCDC buck converter lm2596:XH 2.54mm 3p smd vertical header, F.Cu at (208.1, 131.6)
- added R14: 10K, Resistor_SMD:R_1206_3216Metric, F.Cu at (191.7, 99.3)
- added R15: 10K, Resistor_SMD:R_1206_3216Metric, F.Cu at (191.7, 96.6)
- added R20: 10K, Resistor_SMD:R_1206_3216Metric, F.Cu at (105.7, 99.9)
- added R21: R, Resistor_SMD:R_1206_3216Metric, F.Cu at (185.8, 97.0)
- added R22: R, Resistor_SMD:R_1206_3216Metric, F.Cu at (204.7, 106.6)
- added TH1: Thermistor, Resistor_THT:R_Axial_DIN0204_L3.6mm_D1.6mm_P7.62mm_Horizontal, F.Cu at (105.7, 87.9)
- added U11: MT3608, Package_TO_SOT_SMD:SOT-23-6, F.Cu at (-95.6, 67.0)
- J1: value Conn_01x04_Socket -> PWR LOAD OUT; footprint Connector_JST:JST_GH_SM04B-GHS-TB_1x04-1MP_P1.25mm_Horizontal -> DCDC buck converter lm2596:XH 2.54mm 4p vertical header
- R5: value 1.8K -> 1.2K
- U2: value ~ -> AOD409
- moved A1 135.8 mm to (-56.4, 104.3)
- moved J2 135.8 mm to (-86.8, 58.5)
- moved J3 135.8 mm to (-79.3, 59.8)
- moved Q5 135.8 mm to (-76.1, 92.0)
- moved R13 135.8 mm to (-76.5, 95.9)
- moved R3 135.8 mm to (-76.5, 99.2)
- moved U10 135.8 mm to (-80.6, 104.8)
- moved U9 135.8 mm to (-82.6, 97.8)
- moved R5 59.2 mm to (197.9, 116.2), turned to 180 degrees
- moved REF** 57.5 mm to (219.3, 139.7)
- moved Q3 57.5 mm to (174.5, 140.0)
- moved R2 57.5 mm to (155.1, 127.8)
- moved C1 57.5 mm to (160.0, 129.4)
- moved D1 57.5 mm to (156.4, 131.7)
- moved L1 57.5 mm to (158.9, 137.7)
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Connections:
- net GND renamed -12V
- J1 pad 4: unconnected-(J1-Pin_4-Pad4) -> VD
- J3 pad 2: VD -> unconnected-(J3-Pin_2-Pad2)
- Q4 pad 1: Net-(Q4-G) -> VD
- Q4 pad 3: +VDC -> +12V
- R13 pad 1: Net-(Q5-C) -> Net-(R13-Pad1)
- R13 pad 2: Net-(U10-S) -> Net-(U8-OUT+)
- R5 pad 1: +VDC -> VD
- R5 pad 2: Net-(Q4-G) -> +12V
- SW1 pad 4: Net-(Q1-G) -> Net-(SW1B-A)
- U1 pad 1: +VDC -> +12V
- U7 pad 3: Net-(Q1-G) -> Net-(SW1B-A)
- U9 pad 3: VD -> Net-(U9-IN)
Routing:
- net +VDC: track 75.6 -> 22.0 mm, vias 0 -> 1
- net Net-(SW1B-A): track 0.00 -> 43.6 mm, vias 0 -> 2
- net +12V: track 0.00 -> 38.4 mm
- net Net-(Q1-G): track 45.2 -> 9.23 mm, vias 2 -> 0
- net VD: track 0.00 -> 29.9 mm
- net -12V: track 287.5 -> 314.8 mm
- net OUT 9V+ : track 10.2 -> 27.2 mm
- net -BATT: track 127.3 -> 113.3 mm, vias 2 -> 1
- net Net-(B8-B1+): track 151.4 -> 165.3 mm, vias 0 -> 2
- net Net-(B5-B1-): track 118.1 -> 109.3 mm
- net Net-(D4-A): track 0.00 -> 8.17 mm
- net Net-(Q4-G): track 7.74 -> 0.00 mm
- net Net-(B6-B1+): track 73.8 -> 67.8 mm
- net Net-(U4-P0): track 80.5 -> 86.0 mm
- net Net-(B7-B1+): track 223.5 -> 228.5 mm
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- added copper zone on B.Cu, net +9V
- removed copper zone on B.Cu, net -12V
Other:
- board size 246.6 x 98.4 mm -> 326.2 x 94.7 mm

Commit message: redone bms board and added test bms schem and board to test functionality without the batteries
added:
- bms test schem and layout
- updated bms
- testing of quad rotary encoder breakout board
- testing of teensy audio board
- combining the encoders and audio board in 1 circuit with limited control of chorus fx with encoders
- created text based skeleton structure of GUI of the interface with use of encoders and home button
- created file for adding fx functionality. will be now incorperating fx
Parts:
- removed A1: Arduino_Nano_v3.x, Module:Arduino_Nano
- removed B5, B6, B7, B8: ~, DCDC buck converter lm2596:18650 Batt 2S Holder
- removed C5: 6.2pf, Capacitor_SMD:C_1206_3216Metric
- removed C6: 1uf, Capacitor_SMD:C_1206_3216Metric
- removed D3: ON LED, LED_SMD:LED_1206_3216Metric
- removed DS1: WC1602A, Display:WC1602A
- removed the J2 at (-86.8, 58.5)
- removed the J2 at (209.5, 135.3)
- removed J3: PWR IN, Connector_JST:JST_GH_SM02B-GHS-TB_1x02-1MP_P1.25mm_Horizontal
- removed L1: 10uh, Inductor_SMD:L_6.3x6.3_H3
- removed Q2, Q5: PN100, Package_TO_SOT_SMD:SOT-23
- removed Q3: AO3407, Package_TO_SOT_SMD:SOT-23
- removed R13, R7: 10K, Resistor_SMD:R_1206_3216Metric
- removed R2: 200K, Resistor_SMD:R_1206_3216Metric
- removed R21: R, Resistor_SMD:R_1206_3216Metric
- removed R3, R6: 3k3, Resistor_SMD:R_1206_3216Metric
- removed U10: ~, Package_TO_SOT_SMD:TO-252-2
- removed U11: MT3608, Package_TO_SOT_SMD:SOT-23-6
- removed U9: L78L05_SOT89, Package_TO_SOT_SMD:SOT-89-3
- added B1: ~, DCDC buck converter lm2596:18650 Batt 2S Holder, B.Cu at (97.0, 135.2)
- added B2: ~, DCDC buck converter lm2596:18650 Batt 2S Holder, B.Cu at (143.8, 135.3)
- added B3: ~, DCDC buck converter lm2596:18650 Batt 2S Holder, F.Cu at (71.2, 135.2)
- added B4: ~, DCDC buck converter lm2596:18650 Batt 2S Holder, F.Cu at (143.8, 58.0)
- added C2: C, Capacitor_SMD:C_1206_3216Metric, F.Cu at (207.9, 117.3)
- added J2: B CHG IN, DCDC buck converter lm2596:kf1000 screw terminal, F.Cu at (226.1, 96.0)
- C1: value 4.7uf -> C
- D1: value MBR0530 -> ON LED; footprint Diode_SMD:D_SOD-123 -> LED_SMD:LED_1206_3216Metric
- R1: value 2.2M -> R
- U3: value TPS61040DBV -> L78L05_SOT89; footprint Package_TO_SOT_SMD:SOT-23-5 -> Package_TO_SOT_SMD:SOT-89-3
- moved TP1 113.3 mm to (151.5, 164.8)
- moved TP2 112.4 mm to (151.5, 167.9)
- moved D4 95.2 mm to (144.5, 171.7)
- moved R22 94.3 mm to (135.6, 170.7), turned to 0 degrees
- moved U2 92.9 mm to (138.3, 162.1), turned to 0 degrees
- moved R1 55.5 mm to (208.2, 122.4), turned to 180 degrees
- moved C1 53.3 mm to (208.2, 106.6)
- moved D1 52.0 mm to (208.2, 126.7), turned to 0 degrees
- moved U3 51.9 mm to (207.8, 111.9), turned to 180 degrees
- moved J1 41.1 mm to (228.7, 134.9), turned to 90 degrees
- moved Q4 27.6 mm to (185.3, 133.7), turned to 90 degrees
- moved R5 25.3 mm to (187.1, 139.0), turned to 0 degrees
- moved R9 25.2 mm to (160.1, 115.4), turned to -90 degrees
- moved R10 25.0 mm to (191.1, 134.7), turned to 90 degrees
- moved R15 19.8 mm to (196.2, 115.9), turned to -90 degrees
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Connections:
- C1 pad 2: 5v attiny out -> +BATT
- D1 pad 1: 15v+ CHG VCC -> -12V
- Q1 pad 2: -12V -> -BATT
- Q1 pad 3: -BATT -> -12V
- Q7 pad 3: 15v+ CHG VCC -> +9V
- R1 pad 1: 15v+ CHG VCC -> Net-(U3-OUT)
- R1 pad 2: Net-(U3-FB) -> Net-(D1-A)
- R20 pad 2: Net-(U4-P0) -> Net-(U4-P2)
- R22 pad 1: +VDC -> +BATT
- R9 pad 2: 15v+ CHG VCC -> +9V
- TH1 pad 2: Net-(U4-P0) -> Net-(U4-P2)
- U2 pad 1: +VDC -> CGE SW V+
- U2 pad 3: CGE SW V+ -> +VDC
- U3 pad 1: Net-(D1-A) -> Net-(U3-OUT)
- U3 pad 3: Net-(U3-FB) -> +BATT
- U4 pad 4: Net-(U4-P0) -> Net-(SW1A-B)
- U4 pad 7: Net-(SW1A-B) -> Battery Vref
- U4 pad 8: Battery Vref -> Batt SW VCC
- U4 pad 9: Batt SW VCC -> unconnected-(U4-P5-Pad9)
Routing:
- net Net-(B3-B1+): track 228.5 -> 0.00 mm
- net Net-(B1-B1+): track 212.0 -> 0.00 mm, vias 1 -> 0
- net Net-(B4-B1+): track 165.3 -> 0.00 mm, vias 2 -> 0
- net -12V: track 314.8 -> 168.0 mm, vias 9 -> 5
- net Net-(B1-B1-): track 109.3 -> 0.00 mm, vias 1 -> 0
- net 5v attiny out: track 89.2 -> 0.00 mm
- net Net-(U4-P0): track 86.0 -> 0.00 mm, vias 2 -> 0
- net Battery Vref: track 81.5 -> 3.04 mm
- net CGE SW V+: track 74.5 -> 0.00 mm, vias 2 -> 0
- net Net-(B2-B1+): track 67.8 -> 0.00 mm, vias 1 -> 0
- net -BATT: track 113.3 -> 58.9 mm, vias 1 -> 2
- net 15v+ CHG VCC: track 45.5 -> 0.00 mm
- net Batt SW VCC: track 35.4 -> 0.00 mm
- net +9V: track 80.8 -> 48.4 mm, vias 2 -> 0
- net +12V: track 38.4 -> 7.26 mm
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- removed copper zone on B.Cu, net +9V
Other:
- board size 326.2 x 94.7 mm -> 165.7 x 94.8 mm
- board text removed: "OFF"
- board text removed: "ON"
