File: Research and Development/Interface Section/AFPI/PCB Design/AFPI Device/AFPI Device V1.1/AFPI Device V1.1.kicad_sch (KiCad schematic)
At the start: 28 parts, among them J1 Batt I, J2 OLED, J3 ROT ENC, J4 RGB O, J5 HP O, J6 SP O, J7 AU O, J8 LINE I/PKP V, J9 BACK I, Q1 MPF102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

Commit message: Completed First Revision of AFPI design and Assembly
Finished the initial design and g code generation of the top and bottom plates of the AFPI as well as the central enclosure. couldnt make gcode to fillet the exterior and interior edges as seen on the 3d model as the initial path tools werent enought to do it and i decided on a time scale that the filleted edges werent neccesary for now. if i deem them to be important when designing the guitar body, ill manually dremel fillets and chamfers, however this is not an ideal plan as acrylic is so damn temperamental and brittle.

Currently all packages for the AFPI have arrived and ive already produced the Top and Bottom plates. i took 2 takes for the top plate because the first attempts g code path for the holes used a pocket path which for some reason made the wholes too small. the 7.5mm holes were 6.5, the 3mm were 2.5 and the 2.5mm were ~2.1. when this happened i made the mistake of trying to redrill the holes and i cracked the plate in half on the second hole drilling (there were 16 holes i didnt get very far) on top of this the holes werent accurate circles as the endmill bit would start a bit far out on the edge of each hole.

to remedy this situation i had 3 options,

One would be to file or dremel sand each hole to their correct size, which would be painfully slow and wouldnt actually fix the problem as i would lose much of the advantages that come with a cnc mill being less man hours, accuracy and overall just a more simplistic way of manuafacturing a multi face piece.

The second option would be to use a drill bit to actually drill the holes rather then an endmill bit boring its way in. this wasnt really an option as i didnt want to use specialist bits. even anyway the only 7.5mm bit i could find for a cnc machine was 50$ AUD so no way was i gonna do that for 5 holes, plus i woulld need a 6.5mm as well for the 6.5 hole. The time as well to change each bit and zero the Z probe for each one would just be so time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
Other:
- title: (none) -> AFPI Device V1.1
Changed lines of the file:
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@@
 (kicad_sch (version 20230121) (generator eeschema)
   (paper "A4")
+  (title_block
+    (title "AFPI Device V1.1")
+    (date "2024-08-05")
+  )
   (junction (at 41.91 27.94) (diameter 0) (color 0 0 0 0)
   )
