File: Research and Development/Interface Section/RGB Lighting comps/RGB LED Mounting Board/RGB LED Mounting Board.kicad_pcb (KiCad board)
At the start: 2 copper layers, 84 x 36.8 mm, 26 parts, among them J1 Board 1 In, J2 Board 1 Out, J3 Board 2 In, J4 Board 2 Out

Commit message: Belated Commit of final Files after completed
I actually completed this on the 31/12/2025 however due to  busy new year it was forgotten to commit after the Guitar was completed. Very happy with how it turned out and have many future ideas to include in it.
Parts:
- removed C7, C8: 100nf, Capacitor_SMD:C_1206_3216Metric
- removed D7, D8: WS2812B, LED_SMD:LED_WS2812B_PLCC4_5.0x5.0mm_P3.2mm
- removed J3: Board 2 In, Connector_JST:JST_GH_BM03B-GHS-TBT_1x03-1MP_P1.25mm_Vertical
- removed J4: Board 2 Out, Connector_JST:JST_GH_BM03B-GHS-TBT_1x03-1MP_P1.25mm_Vertical
- removed the REF** at (115.3, 46.8)
- removed the REF** at (193.7, 46.8)
- J1, J2: moved to B.Cu
- moved C6 33.4 mm to (175.8, 20.6), turned to 0 degrees
- moved C5 31.2 mm to (167.5, 20.6), turned to 0 degrees
- moved D6 27.2 mm to (177.0, 25.0), turned to 180 degrees
- moved D5 22.2 mm to (168.7, 25.0), turned to 180 degrees
- moved D4 13.7 mm to (160.4, 25.0)
- moved C4 13.5 mm to (159.2, 20.6)
- moved D3 9.08 mm to (152.1, 25.0)
- moved C3 8.96 mm to (150.8, 20.6)
- moved D2 4.55 mm to (143.8, 25.0)
- moved C2 4.46 mm to (142.5, 20.6)
- moved J2 1.79 mm to (186.6, 26.1), turned to 90 degrees
- moved C9 1.39 mm to (123.3, 21.4), turned to 180 degrees
- moved R1 1.31 mm to (129.3, 27.9)
- turned J1 to 0 degrees
Connections:
- C5 pad 1: GND1 -> GND
- C5 pad 2: VDDA -> VDD
- C6 pad 1: GND1 -> GND
- C6 pad 2: VDDA -> VDD
- D5 pad 1: VDDA -> VDD
- D5 pad 3: GND1 -> GND
- D5 pad 4: Net-(D5-DIN) -> Net-(D4-DOUT)
- D6 pad 1: VDDA -> VDD
- D6 pad 3: GND1 -> GND
- J2 pad 2: Net-(D4-DOUT) -> Net-(D6-DOUT)
Routing:
- net VDDA: track 111.3 -> 0.00 mm
- net GND: track 9.61 -> 44.8 mm, vias 0 -> 2
- net Net-(D5-DIN): track 13.2 -> 0.00 mm
- net Net-(D8-DOUT): track 13.1 -> 0.00 mm
- net VDD: track 115.0 -> 126.8 mm, vias 0 -> 2
- net Net-(D7-DOUT): track 9.32 -> 0.00 mm
- net Net-(D4-DOUT): track 13.7 -> 4.77 mm
- net Net-(D3-DOUT): track 9.34 -> 4.77 mm
- net Net-(D5-DOUT): track 9.34 -> 4.77 mm
- net Net-(D1-DOUT): track 9.32 -> 4.77 mm
- net Net-(D2-DOUT): track 9.29 -> 4.77 mm
- net GND1: track 4.25 -> 0.00 mm
- net Net-(D6-DOUT): track 9.34 -> 7.08 mm, vias 0 -> 1
- net Net-(D1-DIN): track 6.38 -> 4.88 mm
- net Net-(J1-Pin_2): track 8.96 -> 9.51 mm, vias 0 -> 1
- removed copper zone on F.Cu, net GND1
Other:
- board size 84 x 36.8 mm -> 84 x 14.9 mm
- board text removed: "B2"
