File: Research and Development/Interface Section/RGB Lighting comps/RGB LED Mounting Board/RGB LED Mounting Board.kicad_sch (KiCad schematic)
At the start: 22 parts, among them J1 Board 1 In, J2 Board 1 Out, J3 Board 2 In, J4 Board 2 Out

Commit message: Belated Commit of final Files after completed
I actually completed this on the 31/12/2025 however due to  busy new year it was forgotten to commit after the Guitar was completed. Very happy with how it turned out and have many future ideas to include in it.
Parts:
- removed C7, C8: 100nf, Capacitor_SMD:C_1206_3216Metric, symbol Device:C
- removed D7, D8: WS2812B, LED_SMD:LED_WS2812B_PLCC4_5.0x5.0mm_P3.2mm, symbol LED:WS2812B
- removed J3: Board 2 In, Connector_JST:JST_GH_BM03B-GHS-TBT_1x03-1MP_P1.25mm_Vertical, symbol Connector:Conn_01x03_Pin
- removed J4: Board 2 Out, Connector_JST:JST_GH_BM03B-GHS-TBT_1x03-1MP_P1.25mm_Vertical, symbol Connector:Conn_01x03_Pin
Connections:
- net GND1 is gone; now on net GND: C5.1, C6.1, D5.3 (VSS), D6.3 (VSS)
- net VDDA is gone; now on net VDD: C5.2, C6.2, D5.1 (VDD), D6.1 (VDD)
- net at D4.2 (DOUT): now also D5.4 (DIN); no longer J2.2 (Pin_2)
- net at D6.2 (DOUT): now also J2.2 (Pin_2)
Other:
- moved on the sheet: C5, C6, D5, D6, J2
